File: pcb/mx_master_remake/battery.kicad_sch (KiCad schematic)
At the start: 4 parts, among them U3 MCP73811T-420I_OT, U4 LM66200DRLR

Commit message: First
Parts:
- removed U3: MCP73811T-420I_OT, Charger:SOT-23-5_MC_MCH, symbol Charger:MCP73811T-420I_OT
- added R13, R14: 5.1k, Resistor_SMD:R_0603_1608Metric, symbol Device:R_Small
- added SW1: Power Switch, Button_Switch_SMD:SW_SPDT_PCM12, symbol Switch:SW_SPDT
- added U3: MCP73831-2-OT, Package_TO_SOT_SMD:SOT-23-5, symbol Battery_Management:MCP73831-2-OT
Connections:
- net BAT+: now also SW1.3 (C), U3.3 (V_{BAT})
- net GND: now also C1.1, R13.1, R14.2, SW1.1 (A), U3.2 (V_{SS}); no longer C1.2, U4.4 (ON)
- net VBUS: now also C1.2, U3.4 (V_{DD}); no longer C1.1
- new net: SW1.2 (B), U4.4 (ON)
- new net: R13.2, R14.1, U3.5 (PROG)
- new net STAT: U3.1 (STAT)
