File: pcb/mx_master_remake/components.kicad_sch (KiCad schematic)
At the start: 22 parts, among them J5 Daughter Boards, J6 LMB, J7 Mouse Wheel, SW1 BTN_BOTTOM, SW2 BTN_WHEEL, SW3 RMB, U10 MIC2860-2PYD6-TR, U11 MIC2860-2PYD6-TR, U12 MIC2860-2PYD6-TR

Commit message: First
Parts:
- added C16: 0.1uF, Capacitor_SMD:C_0603_1608Metric, symbol Device:C_Small
- renumbered SW1 to SW2, SW2 to SW3, SW3 to SW4
Connections:
- net GND: now also C16.2
- net LMB: now also C16.1
Changed lines of the file:
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@@
     (effects (font (size 1.27 1.27)) (justify left))
+  )
+  (hierarchical_label "LMB" (shape output) (at 236.22 121.92 180) (fields_autoplaced)
+    (effects (font (size 1.27 1.27)) (justify right))
   )
   (hierarchical_label "VBAT" (shape input) (at 88.9 109.22 180) (fields_autoplaced)
@@
   (symbol (lib_id "Switch:SW_Push") (at 193.04 85.09 0) (unit 1)
     (in_bom yes) (on_board yes) (dnp no) (fields_autoplaced)
-    (property "Reference" "SW1" (at 193.04 77.47 0)
+    (property "Reference" "SW2" (at 193.04 77.47 0)
       (effects (font (size 1.27 1.27)))
     )
@@
       (project "mx_master_remake"
         (path "/9f33ee32-6710-4e85-aa53-7616de099ddc/9fc647be-1efb-465b-ba45-8835cb03c883"
-          (reference "SW1") (unit 1)
+          (reference "SW2") (unit 1)
         )
       )
@@
         (path "/9f33ee32-6710-4e85-aa53-7616de099ddc/9fc647be-1efb-465b-ba45-8835cb03c883"
           (reference "#PWR056") (unit 1)
+        )
+      )
+    )
+  )
+  (symbol (lib_id "Device:C_Small") (at 238.76 121.92 90) (unit 1)
+    (in_bom yes) (on_board yes) (dnp no)
+    (property "Reference" "C16" (at 241.3 119.38 90)
+      (effects (font (size 1.27 1.27)))
+    )
+    (property "Value" "0.1uF" (at 236.22 119.38 90)
+      (effects (font (size 1.27 1.27)))
+    )
+    (property "Footprint" "Capacitor_SMD:C_0603_1608Metric" (at 238.76 121.92 0)
+      (effects (font (size 1.27 1.27)) hide)
+    )
+    (property "Datasheet" "~" (at 238.76 121.92 0)
+      (effects (font (size 1.27 1.27)) hide)
+    )
+    (pin "1")
+    (pin "2")
+    (instances
+      (project "mx_master_remake"
+        (path "/9f33ee32-6710-4e85-aa53-7616de099ddc/9fc647be-1efb-465b-ba45-8835cb03c883"
+          (reference "C16") (unit 1)
         )
       )
@@
         (path "/9f33ee32-6710-4e85-aa53-7616de099ddc/9fc647be-1efb-465b-ba45-8835cb03c883"
           (reference "#PWR034") (unit 1)
+        )
+      )
+    )
+  )
+  (symbol (lib_id "power:GND") (at 241.3 121.92 90) (unit 1)
+    (in_bom yes) (on_board yes) (dnp no) (fields_autoplaced)
+    (property "Reference" "#PWR057" (at 247.65 121.92 0)
+      (effects (font (size 1.27 1.27)) hide)
+    )
+    (property "Value" "GND" (at 245.11 121.9199 90)
+      (effects (font (size 1.27 1.27)) (justify right))
+    )
+    (property "Footprint" "" (at 241.3 121.92 0)
+      (effects (font (size 1.27 1.27)) hide)
+    )
+    (property "Datasheet" "" (at 241.3 121.92 0)
+      (effects (font (size 1.27 1.27)) hide)
+    )
+    (pin "1")
+    (instances
+      (project "mx_master_remake"
+        (path "/9f33ee32-6710-4e85-aa53-7616de099ddc/9fc647be-1efb-465b-ba45-8835cb03c883"
+          (reference "#PWR057") (unit 1)
         )
       )
@@
   (symbol (lib_id "Switch:SW_Push") (at 193.04 97.79 0) (unit 1)
     (in_bom yes) (on_board yes) (dnp no) (fields_autoplaced)
-    (property "Reference" "SW2" (at 193.04 90.17 0)
+    (property "Reference" "SW3" (at 193.04 90.17 0)
       (effects (font (size 1.27 1.27)))
     )
@@
       (project "mx_master_remake"
         (path "/9f33ee32-6710-4e85-aa53-7616de099ddc/9fc647be-1efb-465b-ba45-8835cb03c883"
-          (reference "SW2") (unit 1)
+          (reference "SW3") (unit 1)
         )
       )
@@
   (symbol (lib_id "Switch:SW_Push") (at 193.04 110.49 0) (unit 1)
     (in_bom yes) (on_board yes) (dnp no) (fields_autoplaced)
-    (property "Reference" "SW3" (at 193.04 102.87 0)
+    (property "Reference" "SW4" (at 193.04 102.87 0)
       (effects (font (size 1.27 1.27)))
     )
@@
       (project "mx_master_remake"
         (path "/9f33ee32-6710-4e85-aa53-7616de099ddc/9fc647be-1efb-465b-ba45-8835cb03c883"
-          (reference "SW3") (unit 1)
-        )
-      )
+          (reference "SW4") (unit 1)
+        )
+      )
