File: pcb/mx_master_remake/magnet.kicad_sch (KiCad schematic)
At the start: 16 parts, among them U5 AP3012, U6 DGD05473FN-7, U7 DGD05473FN-7, U8 SSM6N7002KFU_LF, U9 SSM6N7002KFU_LF

Commit message: First
Parts:
- L1: footprint Inductor_SMD:L_0603_1608Metric -> Inductor:IND_ASPI-4030S_ABR-L
Connections:
- net +5V: no longer U6.6 (EN), U7.6 (EN)
- new net +3V0: U6.6 (EN), U7.6 (EN)
Changed lines of the file:
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@@
   (junction (at 93.98 78.74) (diameter 0) (color 0 0 0 0)
   )
-  (junction (at 187.96 78.74) (diameter 0) (color 0 0 0 0)
-  )
   (junction (at 134.62 78.74) (diameter 0) (color 0 0 0 0)
   )
@@
   (junction (at 59.69 78.74) (diameter 0) (color 0 0 0 0)
   )
+  (junction (at 193.04 114.3) (diameter 0) (color 0 0 0 0)
+  )
+  (junction (at 193.04 78.74) (diameter 0) (color 0 0 0 0)
+  )
   (junction (at 240.03 81.28) (diameter 0) (color 0 0 0 0)
   )
   (junction (at 147.32 73.66) (diameter 0) (color 0 0 0 0)
   )
-  (junction (at 187.96 114.3) (diameter 0) (color 0 0 0 0)
-  )
   (junction (at 83.82 78.74) (diameter 0) (color 0 0 0 0)
   )
@@
     (stroke (width 0) (type default))
   )
+  (wire (pts (xy 182.88 78.74) (xy 193.04 78.74))
+    (stroke (width 0) (type default))
+  )
   (wire (pts (xy 149.86 78.74) (xy 134.62 78.74))
     (stroke (width 0) (type default))
@@
     (stroke (width 0) (type default))
   )
-  (wire (pts (xy 193.04 78.74) (xy 187.96 78.74))
-    (stroke (width 0) (type default))
-  )
   (wire (pts (xy 102.87 78.74) (xy 106.68 78.74))
     (stroke (width 0) (type default))
@@
     (stroke (width 0) (type default))
   )
-  (wire (pts (xy 185.42 81.28) (xy 185.42 86.36))
+  (wire (pts (xy 187.96 81.28) (xy 187.96 86.36))
     (stroke (width 0) (type default))
   )
@@
     (stroke (width 0) (type default))
   )
-  (wire (pts (xy 182.88 81.28) (xy 185.42 81.28))
-    (stroke (width 0) (type default))
-  )
-  (wire (pts (xy 182.88 116.84) (xy 185.42 116.84))
+  (wire (pts (xy 182.88 81.28) (xy 187.96 81.28))
+    (stroke (width 0) (type default))
+  )
+  (wire (pts (xy 182.88 116.84) (xy 187.96 116.84))
     (stroke (width 0) (type default))
   )
@@
     (stroke (width 0) (type default))
   )
-  (wire (pts (xy 182.88 78.74) (xy 187.96 78.74))
+  (wire (pts (xy 182.88 114.3) (xy 193.04 114.3))
     (stroke (width 0) (type default))
   )
@@
     (stroke (width 0) (type default))
   )
-  (wire (pts (xy 185.42 116.84) (xy 185.42 121.92))
+  (wire (pts (xy 187.96 116.84) (xy 187.96 121.92))
     (stroke (width 0) (type default))
   )
@@
     (stroke (width 0) (type default))
   )
-  (wire (pts (xy 193.04 114.3) (xy 187.96 114.3))
-    (stroke (width 0) (type default))
-  )
   (wire (pts (xy 127 78.74) (xy 134.62 78.74))
     (stroke (width 0) (type default))
   )
-  (wire (pts (xy 187.96 78.74) (xy 187.96 92.71))
+  (wire (pts (xy 193.04 78.74) (xy 193.04 92.71))
     (stroke (width 0) (type default))
   )
@@
     (stroke (width 0) (type default))
   )
-  (wire (pts (xy 185.42 121.92) (xy 195.58 121.92))
+  (wire (pts (xy 187.96 121.92) (xy 195.58 121.92))
     (stroke (width 0) (type default))
   )
@@
     (stroke (width 0) (type default))
   )
-  (wire (pts (xy 187.96 92.71) (xy 240.03 92.71))
+  (wire (pts (xy 193.04 92.71) (xy 240.03 92.71))
     (stroke (width 0) (type default))
   )
@@
     (stroke (width 0) (type default))
   )
-  (wire (pts (xy 185.42 86.36) (xy 195.58 86.36))
+  (wire (pts (xy 187.96 86.36) (xy 195.58 86.36))
     (stroke (width 0) (type default))
   )
@@
     (stroke (width 0) (type default))
   )
-  (wire (pts (xy 182.88 114.3) (xy 187.96 114.3))
-    (stroke (width 0) (type default))
-  )
   (wire (pts (xy 66.04 109.22) (xy 66.04 106.68))
     (stroke (width 0) (type default))
@@
     (stroke (width 0) (type default))
   )
-  (wire (pts (xy 187.96 128.27) (xy 240.03 128.27))
+  (wire (pts (xy 193.04 128.27) (xy 240.03 128.27))
     (stroke (width 0) (type default))
   )
@@
     (stroke (width 0) (type default))
   )
-  (wire (pts (xy 187.96 114.3) (xy 187.96 128.27))
+  (wire (pts (xy 193.04 114.3) (xy 193.04 128.27))
     (stroke (width 0) (type default))
   )
@@
     )
   )
+  (symbol (lib_id "power:+3V0") (at 127 81.28 90) (unit 1)
+    (in_bom yes) (on_board yes) (dnp no) (fields_autoplaced)
+    (property "Reference" "#PWR023" (at 130.81 81.28 0)
+      (effects (font (size 1.27 1.27)) hide)
+    )
+    (property "Value" "+3V0" (at 123.19 81.28 90)
+      (effects (font (size 1.27 1.27)) (justify left))
+    )
+    (property "Footprint" "" (at 127 81.28 0)
+      (effects (font (size 1.27 1.27)) hide)
+    )
+    (property "Datasheet" "" (at 127 81.28 0)
+      (effects (font (size 1.27 1.27)) hide)
+    )
+    (pin "1")
+    (instances
+      (project "mx_master_remake"
+        (path "/9f33ee32-6710-4e85-aa53-7616de099ddc/9cd1b95f-e3f4-4602-b132-130565c9a07e"
+          (reference "#PWR023") (unit 1)
+        )
+      )
+    )
+  )
   (symbol (lib_id "power:GND") (at 231.14 121.92 90) (unit 1)
     (in_bom yes) (on_board yes) (dnp no) (fields_autoplaced)
@@
       (effects (font (size 1.27 1.27)))
     )
-    (property "Footprint" "Inductor_SMD:L_0603_1608Metric" (at 66.04 78.74 0)
-      (effects (font (size 1.27 1.27)) hide)
-    )
-    (property "Datasheet" "~" (at 66.04 78.74 0)
+    (property "Footprint" "Inductor:IND_ASPI-4030S_ABR-L" (at 66.04 78.74 0)
+      (effects (font (size 1.27 1.27)) hide)
+    )
+    (property "Datasheet" "https://www.digikey.com/en/products/detail/abracon-llc/ASPI-4030S-100M-T/4215200" (at 66.04 78.74 0)
       (effects (font (size 1.27 1.27)) hide)
     )
@@
         )
       )
-    )
-  )
-  (symbol (lib_id "power:+5V") (at 127 81.28 90) (unit 1)
-    (in_bom yes) (on_board yes) (dnp no) (fields_autoplaced)
-    (property "Reference" "#PWR023" (at 130.81 81.28 0)
-      (effects (font (size 1.27 1.27)) hide)
-    )
-    (property "Value" "+5V" (at 123.19 81.2799 90)
-      (effects (font (size 1.27 1.27)) (justify left))
-    )
-    (property "Footprint" "" (at 127 81.28 0)
-      (effects (font (size 1.27 1.27)) hide)
-    )
-    (property "Datasheet" "" (at 127 81.28 0)
-      (effects (font (size 1.27 1.27)) hide)
-    )
-    (pin "1")
-    (instances
-      (project "mx_master_remake"
-        (path "/9f33ee32-6710-4e85-aa53-7616de099ddc/9cd1b95f-e3f4-4602-b132-130565c9a07e"
-          (reference "#PWR023") (unit 1)
-        )
-      )
