File: pcb/mx_master_remake/mx_master_remake.kicad_pcb (KiCad board)
At the start: 2 copper layers, 45.9 x 96 mm, 76 parts, among them J1 SWD, J2 Battery, J3 Wheel Magnet, J4 USB4105-GF-A, J5 Daughter Boards, J6 LMB, J7 Mouse Wheel, SW1 BTN_BOTTOM, SW2 BTN_WHEEL, SW3 RMB, SW4 Power Switch, U1 BT840, U10 MIC2860-2PYD6-TR, U11 MIC2860-2PYD6-TR, U12 MIC2860-2PYD6-TR, U13 PAW3370, U14 MIC5501-3.0YM5, U15 TPS613222ADBVR, U16 TLV62568DBVR, U2 D3V3F4U6S-7, U3 MCP73811T-420I_OT, U4 LM66200DRLR, U5 AP3012, U6 DGD05473FN-7, U7 DGD05473FN-7, U8 SSM6N7002KFU_LF, U9 SSM6N7002KFU_LF

Commit message: First
Parts:
- removed the SW4 at (146.6, 77.3)
- added C16: 0.1uF, Capacitor_SMD:C_0603_1608Metric, F.Cu at (136.6, 86.2)
- added R13: 5.1k, Resistor_SMD:R_0603_1608Metric, F.Cu at (161.8, 132.6)
- added R14: 5.1k, Resistor_SMD:R_0603_1608Metric, F.Cu at (160.3, 135.0)
- added SW1: Power Switch, Button_Switch_SMD:SW_SPDT_PCM12, B.Cu at (146.6, 77.3)
- C18: renamed from C17; value 4.7uF/10V -> 10uF/10V
- C24: renamed from C23; value 4.7uF -> 10uF
- C25: renamed from C24; value 4.7uF -> 10uF
- C26: renamed from C25; value 4.7uF -> 10uF
- C27: renamed from C26; value 4.7uF -> 10uF
- C28: renamed from C27; value 22uF -> 10uF
- J4: value USB4105-GF-A -> USB4085-GF-A_REVB; footprint USBC:GCT_USB4105-GF-A -> USBC:GCT_USB4085-GF-A_REVB
- L1: footprint Inductor_SMD:L_0603_1608Metric -> Inductor:IND_ASPI-4030S_ABR-L
- L2: value 2.2uH -> 1uH; footprint Inductor_SMD:L_0603_1608Metric -> Inductor_SMD:L_0805_2012Metric
- L3: footprint Inductor_SMD:L_0603_1608Metric -> Inductor_SMD:L_0805_2012Metric
- U3: value MCP73811T-420I_OT -> MCP73831-2-OT; footprint Charger:SOT-23-5_MC_MCH -> Package_TO_SOT_SMD:SOT-23-5
- moved C12 108.7 mm to (169.6, 118.2), turned to 90 degrees
- moved C11 108.4 mm to (169.6, 114.9), turned to 90 degrees
- moved C10 108.1 mm to (169.6, 111.6), turned to 90 degrees
- moved C9 107.8 mm to (169.6, 108.3), turned to 90 degrees
- moved C7 96.3 mm to (166.4, 98.9), turned to 90 degrees
- moved C6 96.2 mm to (166.4, 109.0), turned to -90 degrees
- moved C5 96.0 mm to (166.4, 102.2), turned to -90 degrees
- moved C13 95.1 mm to (150.0, 128.3)
- moved C8 92.5 mm to (166.4, 105.7), turned to 90 degrees
- moved R8 91.8 mm to (151.8, 125.6), turned to 90 degrees
- moved R7 91.1 mm to (151.8, 121.7), turned to 90 degrees
- moved R6 90.3 mm to (151.8, 117.8), turned to 90 degrees
- moved C15 90.0 mm to (164.3, 70.5)
- moved U8 85.0 mm to (163.3, 97.5), turned to 180 degrees
- moved U9 84.8 mm to (163.3, 104.3), turned to 180 degrees
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- renumbered C16 to C17, C18 to C19, C19 to C20, C20 to C21, C21 to C22, C22 to C23, C28 to C29, SW1 to SW2, SW2 to SW3, SW3 to SW4
Connections:
- net /SWDCLK renamed Net-(J1-SWCLK/TCK)
- net /SWDIO renamed Net-(J1-SWDIO/TMS)
- net /SWO renamed Net-(J1-SWO/TDO)
- net /~{RESET} renamed Net-(J1-~{RESET})
- C1 pad 1: /Battery Management/VBUS -> GND
- C1 pad 2: GND -> /Battery Management/VBUS
- C24 pad 1: Net-(SW4-A) -> /Battery Management/VOUT
- C25 pad 1: Net-(SW4-A) -> /Battery Management/VOUT
- C26 pad 1: Net-(SW4-A) -> /Battery Management/VOUT
- L2 pad 1: Net-(SW4-A) -> /Battery Management/VOUT
- R1 pad 1: GND -> Net-(J4-CC2)
- R1 pad 2: Net-(J4-CC1) -> GND
- R2 pad 1: Net-(J4-CC2) -> GND
- R2 pad 2: GND -> Net-(J4-CC1)
- U1 pad 1: /Sensor/SCLK -> /Magnet/30V_EN
- U1 pad 11: /Mouse Components/BTN_BOTTOM -> /Mouse Components/LMB
- U1 pad 13: /Mouse Components/BTN_BACK -> /Mouse Components/BTN_WHEEL
- U1 pad 2: /Sensor/MOSI -> /Mouse Components/BTN_TOP
- U1 pad 3: /Mouse Components/MW_SCLK -> /Mouse Components/THUMB_LED_1
- U1 pad 4: /Mouse Components/MW_MOSI -> /Mouse Components/THUMB_LED_2
- U1 pad 5: /Mouse Components/MW_MISO -> /Mouse Components/TW_SDA
- U1 pad 6: /Mouse Components/MW_CS -> /Mouse Components/TW_SCL
- U1 pad 7: unconnected-(U1-P0.09/NFC1-Pad7) -> /Mouse Components/TW_RDY
- U1 pad 8: /Mouse Components/BTN_TOP -> /Mouse Components/BTN_BOTTOM
- U1 pad A1: /Sensor/MISO -> unconnected-(U1-P0.28/AIN4-PadA1)
- U1 pad A2: /Sensor/~{NCS} -> unconnected-(U1-P0.29/AIN5-PadA2)
- U1 pad A3: /Mouse Components/MW_INT -> unconnected-(U1-P0.04/AIN2-PadA3)
- U1 pad A5: /Mouse Components/TW_SCL -> /Magnet/NEG
- U1 pad A6: unconnected-(U1-P1.08-PadA6) -> /Mouse Components/BOTTOM_LED_3
- U1 pad B2: /Sensor/~{NRESET} -> unconnected-(U1-P0.30/AIN6-PadB2)
- U1 pad B3: /Sensor/MOTION -> unconnected-(U1-P0.31/AIN7-PadB3)
- U1 pad B4: /Mouse Components/TW_RDY -> unconnected-(U1-P0.06-PadB4)
- U1 pad B5: /Mouse Components/TW_SDA -> /Magnet/POS
- U1 pad B6: unconnected-(U1-P1.03-PadB6) -> /Mouse Components/BTN_BACK
- U1 pad C1: /Mouse Components/BOTTOM_LED_1 -> unconnected-(U1-P0.24-PadC1)
- U1 pad C2: /Mouse Components/BOTTOM_LED_3 -> /Sensor/SCLK
- U1 pad C3: /Mouse Components/LMB -> unconnected-(U1-P0.17-PadC3)
- U1 pad C4: /Mouse Components/BTN_WHEEL -> unconnected-(U1-P0.15-PadC4)
- U1 pad C5: unconnected-(U1-P1.02-PadC5) -> /Mouse Components/BOTTOM_LED_1
- U1 pad C6: unconnected-(U1-P1.04-PadC6) -> /Mouse Components/BOTTOM_LED_2
- U1 pad D1: /Mouse Components/BOTTOM_LED_2 -> /Sensor/MISO
- U1 pad D2: /Mouse Components/THUMB_LED_2 -> /Sensor/MOSI
- U1 pad D3: /Mouse Components/RMB -> /Sensor/~{NCS}
- U1 pad D4: /Mouse Components/BTN_THUMB -> /Mouse Components/MW_INT
- U1 pad D5: unconnected-(U1-P1.01-PadD5) -> /Mouse Components/MW_MOSI
- U1 pad D6: unconnected-(U1-P1.05-PadD6) -> /Mouse Components/MW_CS
- U1 pad E0: unconnected-(U1-P1.07-PadE0) -> /Sensor/MOTION
- U1 pad E1: /Mouse Components/THUMB_LED_1 -> /Sensor/~{NRESET}
- U1 pad E2: unconnected-(U1-P0.21-PadE2) -> /Mouse Components/RMB
- U1 pad E3: unconnected-(U1-P1.09-PadE3) -> /Mouse Components/MW_MISO
- U1 pad E6: /Mouse Components/BTN_FORWARD -> /Mouse Components/MW_SCLK
- U1 pad Z2: /Magnet/POS -> unconnected-(U1-P1.13-PadZ2)
- U1 pad Z3: /Magnet/30V_EN -> unconnected-(U1-P1.14-PadZ3)
- U1 pad Z4: /Magnet/NEG -> /Battery Management/STAT
- U1 pad Z5: unconnected-(U1-P1.10-PadZ5) -> /Mouse Components/BTN_THUMB
- U1 pad Z6: unconnected-(U1-P1.06-PadZ6) -> /Mouse Components/BTN_FORWARD
- U14 pad 1: Net-(SW4-A) -> /Battery Management/VOUT
- U14 pad 3: Net-(SW4-A) -> /Battery Management/VOUT
- U16 pad 1: Net-(SW4-A) -> /Battery Management/VOUT
- U16 pad 4: Net-(SW4-A) -> /Battery Management/VOUT
- U3 pad 1: /Battery Management/VBUS -> /Battery Management/STAT
- U3 pad 5: /Battery Management/VBUS -> Net-(U3-PROG)
- U4 pad 4: GND -> Net-(SW1-B)
- U6 pad 6: +5V -> +3V0
- U7 pad 6: +5V -> +3V0
Routing:
- net /VBAT: track 0.00 -> 109.1 mm, vias 0 -> 10
- net /Magnet/30v: track 0.00 -> 91.0 mm, vias 0 -> 21
- net /Battery Management/VBUS: track 0.00 -> 84.1 mm, vias 0 -> 4
- net GND: track 0.00 -> 72.4 mm, vias 0 -> 86
- net /USB/D+: track 0.00 -> 66.7 mm, vias 0 -> 2
- net /Mouse Components/RMB: track 0.00 -> 66.0 mm, vias 0 -> 2
- net /USB/D-: track 0.00 -> 64.9 mm, vias 0 -> 2
- net +5V: track 0.00 -> 64.6 mm, vias 0 -> 4
- net Net-(SW1-B): track 0.00 -> 58.4 mm, vias 0 -> 2
- net Net-(J1-~{RESET}): track 0.00 -> 56.9 mm, vias 0 -> 2
- net Net-(J1-SWDIO/TMS): track 0.00 -> 55.9 mm, vias 0 -> 2
- net Net-(J1-SWCLK/TCK): track 0.00 -> 54.7 mm, vias 0 -> 2
- net Net-(J1-SWO/TDO): track 0.00 -> 54.7 mm, vias 0 -> 2
- net /Magnet/POS: track 0.00 -> 42.6 mm, vias 0 -> 3
- net /Mouse Components/BTN_TOP: track 0.00 -> 42.5 mm, vias 0 -> 2
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- added copper zone on In2.Cu, net +2V0
- added copper zone on F.Cu, net /Magnet/30v
- added copper zone on B.Cu, net GND
- added copper zone on F.Cu, net GND
- added copper zone on In1.Cu, net GND
- added copper zone on In2.Cu, net GND
Other:
- board size 45.9 x 96 mm -> 39.4 x 96 mm
- copper layers 2 -> 4
