File: pcb/mx_master_remake/sensor.kicad_sch (KiCad schematic)
At the start: 10 parts, among them U13 PAW3370

Commit message: First
Parts:
- C18: renamed from C17; value 4.7uF/10V -> 10uF/10V
- renumbered C16 to C17, C18 to C19, C19 to C20, C20 to C21, C21 to C22, C22 to C23
