File: pcb/mx_master_remake/usb.kicad_sch (KiCad schematic)
At the start: 5 parts, among them J4 USB4105-GF-A, U2 D3V3F4U6S-7

Commit message: First
Parts:
- removed J4: USB4105-GF-A, USBC:GCT_USB4105-GF-A, symbol USBC:USB4105-GF-A
- added J4: USB4085-GF-A_REVB, USBC:GCT_USB4085-GF-A_REVB, symbol USBC:USB4085-GF-A_REVB
Connections:
- net D+: now also J4.A6 (DP1), J4.B6 (DP2)
- net D-: now also J4.A7 (DN1), J4.B7 (DN2)
- net GND: now also R1.2, R2.1, J4.A1 (GND), J4.A12 (GND__1), J4.B1 (GND__2), J4.B12 (GND__3), J4.S1 (SHELL), J4.S2 (SHELL__1), J4.S3 (SHELL__2), J4.S4 (SHELL__3); no longer R1.1, R2.2
- net at FB1.1: now also J4.A4 (VBUS), J4.A9 (VBUS__1), J4.B4 (VBUS__2), J4.B9 (VBUS__3)
- new net: J4.A5 (CC1), R2.2
- new net: J4.B5 (CC2), R1.1
Other:
- moved on the sheet: FB1
